File: Hardware/GeneralPurposeAlarmDevicePCB/Battery_Control.kicad_sch (KiCad schematic)
At the start: 16 parts, among them J703 BATT_JST, J703 BATT_Solder, U701 MCP73833

Commit message: PCB design for battery circuitry layout
Parts:
- removed J703: BATT_Solder, Connector_PinSocket_2.54mm:PinSocket_1x02_P2.54mm_Vertical, symbol Connector_Generic:Conn_01x02
- renumbered R110 to R1, R110 to R2
