File: Hardware/GeneralPurposeAlarmDevicePCB/GeneralPurposeAlarmDevicePCB.kicad_pcb (KiCad board)
At the start: 2 copper layers, 137.2 x 83.8 mm, 140 parts, among them J101 Barrel_Jack_Switch_SMT, J102 0.100_2Pin, J103 0.100_2Pin, J105 S04B-XASK-1(LF)(SN)Rev2, J401 RJ12_6P6C_HORZ, J501 USB_B_Micro_Local, J601 22-23-2021, J602 22-23-2021, Q201 MMBT2222A-7-F, Q202 MMBT2222A-7-F, Q203 MMBT2222A-7-F, Q204 MMBT2222A-7-F, Q205 MMBT2222A-7-F, Q301 BSS138, Q601 BSS138, Q602 DNI, T1 JLC_ToolingHole_0576mm, T2 JLC_ToolingHole_0576mm, T3 JLC_ToolingHole_0576mm, U101 LM7805_TO220, U102 PI_ATMEGA328P-AU-InOrder, U301 PCF8574AT_3_518, U302 LCD_20x4_Character-GPAD_SCH_L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, U501 CH340E

Commit message: PCB design for battery circuitry layout
Parts:
- added C702: 10uF, Capacitor_SMD:C_0603_1608Metric_Pad1.08x0.95mm_HandSolder, F.Cu at (167.6, 68.5)
- added D701: ORANGE 0603, LED_SMD:LED_0603_1608Metric, F.Cu at (159.2, 50.8)
- added D702: GREEN 0603, LED_SMD:LED_0603_1608Metric, F.Cu at (156.5, 54.1)
- added D703: RED 0603, LED_SMD:LED_0603_1608Metric_Pad1.05x0.95mm_HandSolder, F.Cu at (162.6, 53.3)
- added D704: PMEG3020EP, Diode_SMD:D_SOD-128, F.Cu at (159.7, 58.4)
- added J701: BATT_JST, Connector_JST:JST_PH_S2B-PH-K_1x02_P2.00mm_Horizontal, F.Cu at (157.5, 68.6)
- added Q302: AOSS32334C, Package_TO_SOT_SMD:SOT-23, F.Cu at (153.3, 60.0)
- added R701: 330R, Resistor_SMD:R_0603_1608Metric_Pad0.98x0.95mm_HandSolder, F.Cu at (167.6, 66.0)
- added R702: 330R, Resistor_SMD:R_0603_1608Metric_Pad0.98x0.95mm_HandSolder, F.Cu at (167.6, 63.4)
- added R703: 330R, Resistor_SMD:R_0603_1608Metric_Pad0.98x0.95mm_HandSolder, F.Cu at (167.6, 60.9)
- added R704: 2K, Resistor_SMD:R_0603_1608Metric_Pad0.98x0.95mm_HandSolder, F.Cu at (167.6, 58.4)
- added R705: 1K, Resistor_SMD:R_0603_1608Metric_Pad0.98x0.95mm_HandSolder, F.Cu at (167.6, 55.9)
- added R706: 150K, Resistor_SMD:R_0603_1608Metric_Pad0.98x0.95mm_HandSolder, F.Cu at (167.6, 53.4)
- added TH701: 10k Therm, Resistor_SMD:R_0603_1608Metric_Pad0.98x0.95mm_HandSolder, F.Cu at (167.6, 50.9)
- added U701: MCP73833, Package_DFN_QFN:DFN-10-1EP_3x3mm_P0.5mm_EP1.7x2.5mm, F.Cu at (151.9, 67.1)
Connections:
- U102 pad 22: unconnected-(U102-Pad22) -> LCD power
Routing:
- net Vin: track 88.2 -> 113.7 mm
- net +5V: track 457.9 -> 458.4 mm
